File: weatherPCB/WeatherPCB.sch (KiCad schematic (older format))
At the start: 2 parts

Commit message: Updates schematic, changed display output a bit
Parts:
- U?: symbol wemos_mini:WeMos_mini -> WeatherPCB-rescue:WeMos_mini-wemos_mini
- U?: symbol WeatherPCB_Components:TFTLCD_ST7735R -> WeatherPCB-rescue:TFTLCD_ST7735R-WeatherPCB_Components
Changed lines of the file:
@@
 EESchema Schematic File Version 4
+LIBS:WeatherPCB-cache
 EELAYER 26 0
 EELAYER END
@@
 $EndDescr
 $Comp
-L wemos_mini:WeMos_mini U?
+L WeatherPCB-rescue:WeMos_mini-wemos_mini U?
 U 1 1 5D654E45
 P 3200 3500
@@
 $EndComp
 $Comp
-L WeatherPCB_Components:TFTLCD_ST7735R U?
+L WeatherPCB-rescue:TFTLCD_ST7735R-WeatherPCB_Components U?
 U 1 1 5D6562B8
 P 1550 3400

Commit message: Updated schematic for backlighting, renamed pins
Parts:
- added 4.7k, 4.7l: R_US, symbol Device:R_US
- added Q?: 2N4401-ND, digikey-footprints:TO-92-3, symbol digikey-kicad-library:2N4401-ND
- added Q?: 2N4403-ND, digikey-footprints:TO-92-3, symbol digikey-kicad-library:2N4403-ND
- U?: symbol WeatherPCB-rescue:WeMos_mini-wemos_mini -> wemos_mini:WeMos_mini
- U?: symbol WeatherPCB-rescue:TFTLCD_ST7735R-WeatherPCB_Components -> WeatherPCB_Components:TFTLCD_ST7735R
Connections:
- net +5V: now reaches U?.1 (5V)
- net +5V: now also U?.1 (GND)
- net at U?.11 (D0): now also U?.7 (LCD_A0/DC)
- net at U?.13 (D6): now also U?.6 (LCD_RESET)
- net GND: now reaches U?.16 (LED-), U?.2 (GND)
- net GND: now also U?.2 (VCC), Q?.1 (E); no longer U?.1 (GND)
- net at U?.3 (D4): no longer U?.6 (LCD_RESET)
- net at U?.4 (D3): now also 4.7k.2; no longer U?.7 (LCD_A0/DC)
- new net: Q?.3 (C), U?.15 (LED+)
- new net: 4.7k.1, Q?.2 (B)
- new net: 4.7l.2, Q?.3 (C)
- new net: 4.7l.1, Q?.2 (B)
- new net +3V3: Q?.1 (E), U?.16 (3.3V)
- no-connect marks 16 -> 14
Other:
- note added: "BUILTIN_LED"
- note added: "Could use only resistor, or single PNP\nFor safety, using both"
- note added: "PIN MAP\nLCD----ESP8266 (Old)\nRESET---D6 (D4)\nCS-----D8\nA0/DC--D0 (D3)\nSDA----D7\nSCL----D5"
- note removed: "PIN MAP\nLCD----ESP8266 (GPIO)\nRESET---D4 (2,LED)\nCS-----D8 (15,SS)\nA0/DC--D3 (0)\nSDA----D7 (13,MOSI)\nSCL----D5 (14,SCK)"
- moved on the sheet: U?

Commit message: Added photoresistor math, display testing example, updated schematic
Parts:
- added C1: 0.1u, symbol Device:C_Small
- added R1: 220, symbol Device:R_US
- added R2: 70-36k, symbol Device:R_PHOTO
- added R3: 10k, symbol Device:R_US
- R123: renamed from 4.7l; value R_US -> 4.7k
- R142: renamed from 4.7k; value R_US -> 4.7k
- gave numbers to parts that had none: 4
Connections:
- wire segments 41 -> 59
- no-connect marks 14 -> 13
Other:
- note added: "Resistor above R_Photo for safety\nCapacitor smooths out ADC voltage"
- moved on the sheet: Q1, Q2, R123, R142

Commit message: Added PIR and button to schematic
Parts:
- added R3: 10k, symbol Device:R_US
- added SW1: SW_Push, symbol Switch:SW_Push
- added U1: PIR_MTN_SNR, symbol WeatherPCB_Components:PIR_MTN_SNR
- renumbered R142 to R1, R1 to R2, R123 to R4, R2 to R5, R3 to R6, U1 to U2, U2 to U3
Connections:
- wire segments 59 -> 71
- no-connect marks 13 -> 11
Other:
- note added: "Smaller model - volt reg side up"
- moved on the sheet: Q1, Q2, R1, R2, R4, R6, U2, U3

Commit message: Reconfigured BJTs on schematic
Connections:
- wire segments 71 -> 73
Other:
- moved on the sheet: Q1, R4
Changed lines of the file:
@@
 Text Notes 4500 3050 0    50   ~ 0
 BUILTIN_LED
-Connection ~ 4600 2750
-Wire Wire Line
-	4600 2750 4600 2800
 $Comp
 L digikey-kicad-library:2N4403-ND Q1
 U 1 1 5D69C8C7
-P 5450 4350
-F 0 "Q1" H 5637 4403 60  0000 L CNN
-F 1 "2N4403-ND" H 5250 4050 60  0000 L CNN
-F 2 "digikey-footprints:TO-92-3" H 5750 4650 60  0001 L CNN
-F 3 "" H 5650 4650 60  0001 L CNN
-	1    5450 4350
+P 5250 4350
+F 0 "Q1" H 5437 4403 60  0000 L CNN
+F 1 "2N4403-ND" H 5050 4050 60  0000 L CNN
+F 2 "digikey-footprints:TO-92-3" H 5550 4650 60  0001 L CNN
+F 3 "" H 5450 4650 60  0001 L CNN
+	1    5250 4350
 	1    0    0    -1
 $EndComp
@@
 L power:+3.3V #PWR011
 U 1 1 5D69E044
-P 5550 4100
-F 0 "#PWR011" H 5550 3950 50  0001 C CNN
-F 1 "+3.3V" H 5565 4273 50  0000 C CNN
-F 2 "" H 5550 4100 50  0001 C CNN
-F 3 "" H 5550 4100 50  0001 C CNN
-	1    5550 4100
+P 5350 3950
+F 0 "#PWR011" H 5350 3800 50  0001 C CNN
+F 1 "+3.3V" H 5365 4123 50  0000 C CNN
+F 2 "" H 5350 3950 50  0001 C CNN
+F 3 "" H 5350 3950 50  0001 C CNN
+	1    5350 3950
 	1    0    0    -1
 $EndComp
@@
 L Device:R_US R4
 U 1 1 5D69E708
-P 5050 4350
-F 0 "R4" V 4845 4350 50  0000 C CNN
-F 1 "4.7k" V 4936 4350 50  0000 C CNN
-F 2 "" V 5090 4340 50  0001 C CNN
-F 3 "~" H 5050 4350 50  0001 C CNN
-	1    5050 4350
-	0    1    1    0
+P 4800 4150
+F 0 "R4" V 4595 4150 50  0000 C CNN
+F 1 "4.7k" V 4686 4150 50  0000 C CNN
+F 2 "" V 4840 4140 50  0001 C CNN
+F 3 "~" H 4800 4150 50  0001 C CNN
+	1    4800 4150
+	-1   0    0    1
 $EndComp
 $Comp
@@
 	4800 4800 4800 4750
 Wire Wire Line
-	5200 4350 5250 4350
-Wire Wire Line
-	5550 4150 5550 4100
-Wire Wire Line
 	4450 3750 4450 3100
 Wire Wire Line
@@
 Wire Wire Line
 	4450 3100 5000 3100
-Wire Wire Line
-	4800 4350 4900 4350
 Wire Wire Line
 	5900 3600 6800 3600
@@
 	5900 3800 5800 3800
 Wire Wire Line
-	5800 3800 5800 4600
-Wire Wire Line
-	5800 4600 5550 4600
-Wire Wire Line
-	5550 4600 5550 4550
+	5350 4600 5350 4550
 $Comp
 L power:+3.3V #PWR08
@@
 	3000 4500 3000 4400
 Wire Wire Line
-	3000 4000 3000 4100
-Wire Wire Line
-	3050 4050 4050 4050
+	3000 4000 3000 4050
 Wire Wire Line
 	4050 4050 4050 3300
@@
 Text Notes 3600 2800 0    30   ~ 0
 Smaller model - volt reg side up
+Wire Wire Line
+	4800 4300 4800 4350
+Wire Wire Line
+	5050 4350 4800 4350
+Connection ~ 4800 4350
+Wire Wire Line
+	5800 3800 5800 4600
+Wire Wire Line
+	5350 4600 5800 4600
+Wire Wire Line
+	5350 4000 5350 4150
+Wire Wire Line
+	4800 4000 5350 4000
+Wire Wire Line
+	5350 3950 5350 4000
+Connection ~ 5350 4000
+Wire Wire Line
+	3000 4050 4050 4050
+Connection ~ 3000 4050
+Wire Wire Line
+	3000 4050 3000 4100
 $EndSCHEMATC

Commit message: Started on PCB
Parts:
- added SW2: SW_SPDT, Pin_Headers:Pin_Header_Straight_1x03_Pitch2.54mm, symbol Switch:SW_SPDT
- C1: footprint (none) -> Capacitors_THT:C_Axial_L3.8mm_D2.6mm_P7.50mm_Horizontal
- Q1, Q2: footprint digikey-footprints:TO-92-3 -> TO_SOT_Packages_THT:TO-92_Inline_Narrow_Oval
- R1, R2, R5, R6: footprint (none) -> Resistors_THT:R_Axial_DIN0204_L3.6mm_D1.6mm_P5.08mm_Horizontal
- R3: renamed from R4; footprint (none) -> Resistors_THT:R_Axial_DIN0204_L3.6mm_D1.6mm_P5.08mm_Horizontal
- R4: renamed from R3; footprint (none) -> Resistors_THT:R_Axial_DIN0204_L3.6mm_D1.6mm_P5.08mm_Horizontal
- SW1: footprint (none) -> Buttons_Switches_THT:SW_PUSH_6mm_h5mm
- U1: footprint (none) -> Pin_Headers:Pin_Header_Angled_1x03_Pitch2.54mm
- U2: footprint (none) -> Modules2:WEMOS_D1_mini_light
- U3: footprint (none) -> Pin_Headers:Pin_Header_Straight_1x16_Pitch2.54mm
Connections:
- net labels added: GNDPWR
- wire segments 73 -> 85
Other:
- moved on the sheet: Q1, Q2, R1, R3, U2

Commit message: created pcb
Parts:
- C1: footprint Capacitors_THT:C_Axial_L3.8mm_D2.6mm_P7.50mm_Horizontal -> Capacitors_THT:C_Disc_D3.8mm_W2.6mm_P2.50mm; Where to Buy (none) -> https://www.digikey.com/product-detail/en/avx-corporation/S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
- Q1, Q2: Where to Buy (none) -> https://www.digikey.com/product-detail/en/micro-commercial-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
- R1, R2, R3, R4, R6: Where to Buy (none) -> https://www.digikey.com/product-detail/en/stackpole-electro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
- R5: Where to Buy (none) -> https://www.amazon.com/GeeBat-Photoresistor-Resistors-Light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
- SW1: Where to Buy (none) -> https://www.digikey.com/product-detail/en/te-connectivity-a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
- SW2: Where to Buy (none) -> https://www.amazon.com/gp/product/B007QAJUUS/
- U1: Where to Buy (none) -> https://www.amazon.com/gp/product/B07LF47TRC
- U2: Where to Buy (none) -> https://www.amazon.com/gp/product/B076F53B6S/
Changed lines of the file:
@@
 F 2 "Modules2:WEMOS_D1_mini_light" H 6050 2600 60  0001 C CNN
 F 3 "https://wiki.wemos.cc/_media/products:d1:sch_d1_mini_v3.0.0.pdf" H 5500 3831 60  0001 C CNN
+F 4 "https://www.amazon.com/gp/product/B076F53B6S/" H 0   0   50  0001 C CNN "Where to Buy"
 	1    5500 3300
 	-1   0    0    1
@@
 F 2 "TO_SOT_Packages_THT:TO-92_Inline_Narrow_Oval" H 4816 4978 60  0001 L CNN
 F 3 "" H 4750 4900 60  0001 L CNN
+F 4 "https://www.digikey.com/product-detail/en/micro-commercial-co/2N4401-AP/2N4401-APCT-ND/950593" H 0   0   50  0001 C CNN "Where to Buy"
 	1    4550 4600
 	1    0    0    -1
@@
 F 2 "TO_SOT_Packages_THT:TO-92_Inline_Narrow_Oval" H 5400 4700 60  0001 L CNN
 F 3 "" H 5300 4700 60  0001 L CNN
+F 4 "https://www.digikey.com/product-detail/en/micro-commercial-co/2N4403-AP/2N4403-APCT-ND/950594" H 0   0   50  0001 C CNN "Where to Buy"
 	1    5100 4400
 	1    0    0    -1
@@
 F 2 "Resistors_THT:R_Axial_DIN0204_L3.6mm_D1.6mm_P5.08mm_Horizontal" V 4690 4190 50  0001 C CNN
 F 3 "~" H 4650 4200 50  0001 C CNN
+F 4 "https://www.digikey.com/product-detail/en/stackpole-electronics-inc/CF14JT4K70/CF14JT4K70CT-ND/1830366" H 0   0   50  0001 C CNN "Where to Buy"
 	1    4650 4200
 	-1   0    0    1
@@
 F 2 "Resistors_THT:R_Axial_DIN0204_L3.6mm_D1.6mm_P5.08mm_Horizontal" V 4340 3940 50  0001 C CNN
 F 3 "~" H 4300 3950 50  0001 C CNN
+F 4 "https://www.digikey.com/product-detail/en/stackpole-electronics-inc/CF14JT4K70/CF14JT4K70CT-ND/1830366" H 0   0   50  0001 C CNN "Where to Buy"
 	1    4300 3950
 	-1   0    0    1
@@
 F 2 "Resistors_THT:R_Axial_DIN0204_L3.6mm_D1.6mm_P5.08mm_Horizontal" V 6140 4140 50  0001 C CNN
 F 3 "~" H 6100 4150 50  0001 C CNN
+F 4 "https://www.digikey.com/product-detail/en/stackpole-electronics-inc/CF14JT220R/CF14JT220RCT-ND/1830334" H 0   0   50  0001 C CNN "Where to Buy"
 	1    6100 4150
 	1    0    0    -1
@@
 F 2 "Resistors_THT:R_Axial_DIN0204_L3.6mm_D1.6mm_P5.08mm_Horizontal" V 6140 4890 50  0001 C CNN
 F 3 "~" H 6100 4900 50  0001 C CNN
+F 4 "https://www.digikey.com/product-detail/en/stackpole-electronics-inc/CF14JT10K0/CF14JT10K0CT-ND/1830374" H 0   0   50  0001 C CNN "Where to Buy"
 	1    6100 4900
 	1    0    0    -1
@@
 F 2 "Resistors_THT:R_Axial_DIN0204_L3.6mm_D1.6mm_P5.08mm_Horizontal" V 6150 4250 50  0001 L CNN
 F 3 "~" H 6100 4450 50  0001 C CNN
+F 4 "https://www.amazon.com/GeeBat-Photoresistor-Resistors-Light-dependen-Optoresistor/dp/B01N0GJ6QP/ref=sr_1_9?keywords=photoresistor&qid=1568421612&sr=8-9" H 0   0   50  0001 C CNN "Where to Buy"
 	1    6100 4500
 	1    0    0    -1
@@
 F 0 "C1" H 6592 4946 50  0000 L CNN
 F 1 "0.1u" H 6592 4855 50  0000 L CNN
-F 2 "Capacitors_THT:C_Axial_L3.8mm_D2.6mm_P7.50mm_Horizontal" H 6500 4900 50  0001 C CNN
+F 2 "Capacitors_THT:C_Disc_D3.8mm_W2.6mm_P2.50mm" H 6500 4900 50  0001 C CNN
 F 3 "~" H 6500 4900 50  0001 C CNN
+F 4 "https://www.digikey.com/product-detail/en/avx-corporation/SR215C104KAR/478-3188-ND/936830" H 0   0   50  0001 C CNN "Where to Buy"
 	1    6500 4900
 	1    0    0    -1
@@
 F 2 "Buttons_Switches_THT:SW_PUSH_6mm_h5mm" H 3000 4000 50  0001 C CNN
 F 3 "" H 3000 4000 50  0001 C CNN
+F 4 "https://www.digikey.com/product-detail/en/te-connectivity-alcoswitch-switches/1825910-6/450-1650-ND/1632536" H 3000 3800 50  0001 C CNN "Where to Buy"
 	1    3000 3800
 	0    1    1    0
@@
 F 2 "Resistors_THT:R_Axial_DIN0204_L3.6mm_D1.6mm_P5.08mm_Horizontal" V 3040 4240 50  0001 C CNN
 F 3 "~" H 3000 4250 50  0001 C CNN
+F 4 "https://www.digikey.com/product-detail/en/stackpole-electronics-inc/CF14JT10K0/CF14JT10K0CT-ND/1830374" H 0   0   50  0001 C CNN "Where to Buy"
 	1    3000 4250
 	1    0    0    -1
@@
 F 2 "Pin_Headers:Pin_Header_Angled_1x03_Pitch2.54mm" H 3400 2500 50  0001 C CNN
 F 3 "" H 3400 2500 50  0001 C CNN
+F 4 "https://www.amazon.com/gp/product/B07LF47TRC" H 0   0   50  0001 C CNN "Where to Buy"
 	1    3400 2500
 	1    0    0    -1
@@
 F 2 "Pin_Headers:Pin_Header_Straight_1x03_Pitch2.54mm" H 5650 4150 50  0001 C CNN
 F 3 "" H 5650 4150 50  0001 C CNN
+F 4 "https://www.amazon.com/gp/product/B007QAJUUS/" H 0   0   50  0001 C CNN "Where to Buy"
 	1    5650 4150
 	-1   0    0    1

Commit message: Rev 1 PCB finished
Parts:
- added H1, H2, H3, H4: MountingHole, Mounting_Holes:MountingHole_2.7mm, symbol Mechanical:MountingHole
- C1: footprint Capacitors_THT:C_Disc_D3.8mm_W2.6mm_P2.50mm -> Capacitors_THT:C_Disc_D3.0mm_W1.6mm_P2.50mm
Changed lines of the file:
@@
 EELAYER 26 0
 EELAYER END
-$Descr A4 11693 8268
+$Descr USLetter 11000 8500
 encoding utf-8
 Sheet 1 1
@@
 F 0 "C1" H 6592 4946 50  0000 L CNN
 F 1 "0.1u" H 6592 4855 50  0000 L CNN
-F 2 "Capacitors_THT:C_Disc_D3.8mm_W2.6mm_P2.50mm" H 6500 4900 50  0001 C CNN
+F 2 "Capacitors_THT:C_Disc_D3.0mm_W1.6mm_P2.50mm" H 6500 4900 50  0001 C CNN
 F 3 "~" H 6500 4900 50  0001 C CNN
 F 4 "https://www.digikey.com/product-detail/en/avx-corporation/SR215C104KAR/478-3188-ND/936830" H 0   0   50  0001 C CNN "Where to Buy"
@@
 Wire Wire Line
 	5900 4150 5850 4150
+$Comp
+L Mechanical:MountingHole H4
+U 1 1 5D803844
+P 7050 6550
+F 0 "H4" H 7150 6596 50  0000 L CNN
+F 1 "MountingHole" H 7150 6505 50  0000 L CNN
+F 2 "Mounting_Holes:MountingHole_2.7mm" H 7050 6550 50  0001 C CNN
+F 3 "~" H 7050 6550 50  0001 C CNN
+	1    7050 6550
+	1    0    0    -1
+$EndComp
+$Comp
+L Mechanical:MountingHole H3
+U 1 1 5D805BF3
+P 7050 6400
+F 0 "H3" H 7150 6446 50  0000 L CNN
+F 1 "MountingHole" H 7150 6355 50  0000 L CNN
+F 2 "Mounting_Holes:MountingHole_2.7mm" H 7050 6400 50  0001 C CNN
+F 3 "~" H 7050 6400 50  0001 C CNN
+	1    7050 6400
+	1    0    0    -1
+$EndComp
+$Comp
+L Mechanical:MountingHole H2
+U 1 1 5D805C29
+P 7050 6250
+F 0 "H2" H 7150 6296 50  0000 L CNN
+F 1 "MountingHole" H 7150 6205 50  0000 L CNN
+F 2 "Mounting_Holes:MountingHole_2.7mm" H 7050 6250 50  0001 C CNN
+F 3 "~" H 7050 6250 50  0001 C CNN
+	1    7050 6250
+	1    0    0    -1
+$EndComp
+$Comp
+L Mechanical:MountingHole H1
+U 1 1 5D805C61
+P 7050 6100
+F 0 "H1" H 7150 6146 50  0000 L CNN
+F 1 "MountingHole" H 7150 6055 50  0000 L CNN
+F 2 "Mounting_Holes:MountingHole_2.7mm" H 7050 6100 50  0001 C CNN
+F 3 "~" H 7050 6100 50  0001 C CNN
+	1    7050 6100
+	1    0    0    -1
+$EndComp
 $EndSCHEMATC
