File: weatherPCB/WeatherPCB.sch (KiCad schematic (older format))
At the start: 18 parts, among them Q1 2N4403-ND, Q2 2N4401-ND, SW1 SW_Push, SW2 SW_SPDT, U1 PIR_MTN_SNR, U2 WeMos_mini, U3 TFTLCD_ST7735R

Commit message: Modified PCB for larger resistor sizes and KiCad error with display wiring
Parts:
- C1: footprint Capacitors_THT:C_Disc_D3.0mm_W1.6mm_P2.50mm -> Capacitors_THT:C_Disc_D7.0mm_W2.5mm_P5.00mm
- R1, R2, R3, R4, R5, R6: footprint Resistors_THT:R_Axial_DIN0204_L3.6mm_D1.6mm_P5.08mm_Horizontal -> Resistors_THT:R_Axial_DIN0204_L3.6mm_D1.6mm_P7.62mm_Horizontal
Changed lines of the file:
@@
 F 0 "R3" V 4445 4200 50  0000 C CNN
 F 1 "4.7k" V 4536 4200 50  0000 C CNN
-F 2 "Resistors_THT:R_Axial_DIN0204_L3.6mm_D1.6mm_P5.08mm_Horizontal" V 4690 4190 50  0001 C CNN
+F 2 "Resistors_THT:R_Axial_DIN0204_L3.6mm_D1.6mm_P7.62mm_Horizontal" V 4690 4190 50  0001 C CNN
 F 3 "~" H 4650 4200 50  0001 C CNN
 F 4 "https://www.digikey.com/product-detail/en/stackpole-electronics-inc/CF14JT4K70/CF14JT4K70CT-ND/1830366" H 0   0   50  0001 C CNN "Where to Buy"
@@
 F 0 "R1" H 4232 3904 50  0000 R CNN
 F 1 "4.7k" H 4232 3995 50  0000 R CNN
-F 2 "Resistors_THT:R_Axial_DIN0204_L3.6mm_D1.6mm_P5.08mm_Horizontal" V 4340 3940 50  0001 C CNN
+F 2 "Resistors_THT:R_Axial_DIN0204_L3.6mm_D1.6mm_P7.62mm_Horizontal" V 4340 3940 50  0001 C CNN
 F 3 "~" H 4300 3950 50  0001 C CNN
 F 4 "https://www.digikey.com/product-detail/en/stackpole-electronics-inc/CF14JT4K70/CF14JT4K70CT-ND/1830366" H 0   0   50  0001 C CNN "Where to Buy"
@@
 F 0 "R2" H 6168 4196 50  0000 L CNN
 F 1 "220" H 6168 4105 50  0000 L CNN
-F 2 "Resistors_THT:R_Axial_DIN0204_L3.6mm_D1.6mm_P5.08mm_Horizontal" V 6140 4140 50  0001 C CNN
+F 2 "Resistors_THT:R_Axial_DIN0204_L3.6mm_D1.6mm_P7.62mm_Horizontal" V 6140 4140 50  0001 C CNN
 F 3 "~" H 6100 4150 50  0001 C CNN
 F 4 "https://www.digikey.com/product-detail/en/stackpole-electronics-inc/CF14JT220R/CF14JT220RCT-ND/1830334" H 0   0   50  0001 C CNN "Where to Buy"
@@
 F 0 "R6" H 6168 4946 50  0000 L CNN
 F 1 "10k" H 6168 4855 50  0000 L CNN
-F 2 "Resistors_THT:R_Axial_DIN0204_L3.6mm_D1.6mm_P5.08mm_Horizontal" V 6140 4890 50  0001 C CNN
+F 2 "Resistors_THT:R_Axial_DIN0204_L3.6mm_D1.6mm_P7.62mm_Horizontal" V 6140 4890 50  0001 C CNN
 F 3 "~" H 6100 4900 50  0001 C CNN
 F 4 "https://www.digikey.com/product-detail/en/stackpole-electronics-inc/CF14JT10K0/CF14JT10K0CT-ND/1830374" H 0   0   50  0001 C CNN "Where to Buy"
@@
 F 0 "R5" H 6170 4546 50  0000 L CNN
 F 1 "70-36k" H 6170 4455 50  0000 L CNN
-F 2 "Resistors_THT:R_Axial_DIN0204_L3.6mm_D1.6mm_P5.08mm_Horizontal" V 6150 4250 50  0001 L CNN
+F 2 "Resistors_THT:R_Axial_DIN0204_L3.6mm_D1.6mm_P7.62mm_Horizontal" V 6150 4250 50  0001 L CNN
 F 3 "~" H 6100 4450 50  0001 C CNN
 F 4 "https://www.amazon.com/GeeBat-Photoresistor-Resistors-Light-dependen-Optoresistor/dp/B01N0GJ6QP/ref=sr_1_9?keywords=photoresistor&qid=1568421612&sr=8-9" H 0   0   50  0001 C CNN "Where to Buy"
@@
 F 0 "C1" H 6592 4946 50  0000 L CNN
 F 1 "0.1u" H 6592 4855 50  0000 L CNN
-F 2 "Capacitors_THT:C_Disc_D3.0mm_W1.6mm_P2.50mm" H 6500 4900 50  0001 C CNN
+F 2 "Capacitors_THT:C_Disc_D7.0mm_W2.5mm_P5.00mm" H 6500 4900 50  0001 C CNN
 F 3 "~" H 6500 4900 50  0001 C CNN
 F 4 "https://www.digikey.com/product-detail/en/avx-corporation/SR215C104KAR/478-3188-ND/936830" H 0   0   50  0001 C CNN "Where to Buy"
@@
 F 0 "R4" H 3068 4296 50  0000 L CNN
 F 1 "10k" H 3068 4205 50  0000 L CNN
-F 2 "Resistors_THT:R_Axial_DIN0204_L3.6mm_D1.6mm_P5.08mm_Horizontal" V 3040 4240 50  0001 C CNN
+F 2 "Resistors_THT:R_Axial_DIN0204_L3.6mm_D1.6mm_P7.62mm_Horizontal" V 3040 4240 50  0001 C CNN
 F 3 "~" H 3000 4250 50  0001 C CNN
 F 4 "https://www.digikey.com/product-detail/en/stackpole-electronics-inc/CF14JT10K0/CF14JT10K0CT-ND/1830374" H 0   0   50  0001 C CNN "Where to Buy"

Commit message: Added space for optional 1-wire temp sensor
Parts:
- added U4: DS1822, TO_SOT_Packages_THT:TO-92_Inline_Wide, symbol Sensor_Temperature:DS1822
- Q1, Q2: footprint TO_SOT_Packages_THT:TO-92_Inline_Narrow_Oval -> TO_SOT_Packages_THT:TO-92_Inline_Wide
Connections:
- wire segments 85 -> 93
- no-connect marks 11 -> 10
Other:
- note added: "OPTIONAL"
- note added: "Optionally, can use 4.7k resistors instead of 10k (or vice versa)."
Changed lines of the file:
@@
 U 1 1 5D654E45
 P 5500 3300
-F 0 "U2" H 5500 3800 60  0000 C CNN
+F 0 "U2" H 5500 3650 60  0000 C CNN
 F 1 "WeMos_mini" H 5500 2650 60  0000 C CNN
 F 2 "Modules2:WEMOS_D1_mini_light" H 6050 2600 60  0001 C CNN
@@
 F 0 "Q2" H 4737 4653 60  0000 L CNN
 F 1 "2N4401-ND" H 4000 4400 60  0000 L CNN
-F 2 "TO_SOT_Packages_THT:TO-92_Inline_Narrow_Oval" H 4816 4978 60  0001 L CNN
+F 2 "TO_SOT_Packages_THT:TO-92_Inline_Wide" H 4816 4978 60  0001 L CNN
 F 3 "" H 4750 4900 60  0001 L CNN
 F 4 "https://www.digikey.com/product-detail/en/micro-commercial-co/2N4401-AP/2N4401-APCT-ND/950593" H 0   0   50  0001 C CNN "Where to Buy"
@@
 	1    0    0    -1
 $EndComp
-NoConn ~ 5000 3000
-Text Notes 4500 3050 0    50   ~ 0
+Text Notes 4750 2975 0    30   ~ 0
 BUILTIN_LED
 $Comp
@@
 F 0 "Q1" H 5287 4453 60  0000 L CNN
 F 1 "2N4403-ND" H 4900 4100 60  0000 L CNN
-F 2 "TO_SOT_Packages_THT:TO-92_Inline_Narrow_Oval" H 5400 4700 60  0001 L CNN
+F 2 "TO_SOT_Packages_THT:TO-92_Inline_Wide" H 5400 4700 60  0001 L CNN
 F 3 "" H 5300 4700 60  0001 L CNN
 F 4 "https://www.digikey.com/product-detail/en/micro-commercial-co/2N4403-AP/2N4403-APCT-ND/950594" H 0   0   50  0001 C CNN "Where to Buy"
@@
 	1    0    0    -1
 $EndComp
+Text Notes 7525 5375 0    50   ~ 0
+Optionally, can use 4.7k resistors instead of 10k (or vice versa).
+$Comp
+L Sensor_Temperature:DS1822 U4
+U 1 1 5DA67D1B
+P 4350 2025
+F 0 "U4" H 4120 2071 50  0000 R CNN
+F 1 "DS1822" H 4120 1980 50  0000 R CNN
+F 2 "TO_SOT_Packages_THT:TO-92_Inline_Wide" H 3350 1775 50  0001 C CNN
+F 3 "http://datasheets.maximintegrated.com/en/ds/DS1822.pdf" H 4200 2275 50  0001 C CNN
+	1    4350 2025
+	1    0    0    -1
+$EndComp
+Wire Wire Line
+	5025 3000 5000 3000
+Wire Wire Line
+	4475 3000 4475 2375
+Wire Wire Line
+	4475 2375 4700 2375
+Wire Wire Line
+	4700 2375 4700 2025
+Wire Wire Line
+	4700 2025 4650 2025
+Connection ~ 5000 3000
+Wire Wire Line
+	5000 3000 4475 3000
+Text Notes 3750 1900 0    50   ~ 0
+OPTIONAL
+$Comp
+L power:GND #PWR0105
+U 1 1 5DA6A555
+P 4350 2375
+F 0 "#PWR0105" H 4350 2125 50  0001 C CNN
+F 1 "GND" H 4355 2202 50  0000 C CNN
+F 2 "" H 4350 2375 50  0001 C CNN
+F 3 "" H 4350 2375 50  0001 C CNN
+	1    4350 2375
+	1    0    0    -1
+$EndComp
+$Comp
+L power:+3.3V #PWR0106
+U 1 1 5DA6A586
+P 4350 1675
+F 0 "#PWR0106" H 4350 1525 50  0001 C CNN
+F 1 "+3.3V" H 4365 1848 50  0000 C CNN
+F 2 "" H 4350 1675 50  0001 C CNN
+F 3 "" H 4350 1675 50  0001 C CNN
+	1    4350 1675
+	1    0    0    -1
+$EndComp
+Wire Wire Line
+	4350 2375 4350 2325
+Wire Wire Line
+	4350 1725 4350 1675
 $EndSCHEMATC

Commit message: Moved parts around on schematic, no part changes
Other:
- note added: "Optionally, can use 4.7k \nresistors instead of 10k \n(or vice versa)."
- note removed: "Optionally, can use 4.7k resistors instead of 10k (or vice versa)."
Changed lines of the file:
@@
 EESchema Schematic File Version 4
 LIBS:WeatherPCB-cache
-EELAYER 26 0
+EELAYER 30 0
 EELAYER END
 $Descr USLetter 11000 8500
@@
 L power:GND #PWR0101
 U 1 1 5D7DAD12
-P 9100 6200
-F 0 "#PWR0101" H 9100 5950 50  0001 C CNN
-F 1 "GND" H 9105 6027 50  0000 C CNN
-F 2 "" H 9100 6200 50  0001 C CNN
-F 3 "" H 9100 6200 50  0001 C CNN
-	1    9100 6200
+P 4270 5410
+F 0 "#PWR0101" H 4270 5160 50  0001 C CNN
+F 1 "GND" H 4275 5237 50  0000 C CNN
+F 2 "" H 4270 5410 50  0001 C CNN
+F 3 "" H 4270 5410 50  0001 C CNN
+	1    4270 5410
 	1    0    0    -1
 $EndComp
@@
 L power:GNDPWR #PWR0102
 U 1 1 5D7DADA4
-P 9350 6200
-F 0 "#PWR0102" H 9350 6000 50  0001 C CNN
-F 1 "GNDPWR" H 9354 6046 50  0000 C CNN
-F 2 "" H 9350 6150 50  0001 C CNN
-F 3 "" H 9350 6150 50  0001 C CNN
-	1    9350 6200
-	1    0    0    -1
-$EndComp
-Wire Wire Line
-	9350 6200 9350 6100
-Wire Wire Line
-	9350 6100 9100 6100
-Wire Wire Line
-	9100 6100 9100 6200
+P 4520 5410
+F 0 "#PWR0102" H 4520 5210 50  0001 C CNN
+F 1 "GNDPWR" H 4524 5256 50  0000 C CNN
+F 2 "" H 4520 5360 50  0001 C CNN
+F 3 "" H 4520 5360 50  0001 C CNN
+	1    4520 5410
+	1    0    0    -1
+$EndComp
+Wire Wire Line
+	4520 5410 4520 5310
+Wire Wire Line
+	4520 5310 4270 5310
+Wire Wire Line
+	4270 5310 4270 5410
 $Comp
 L power:+3.3V #PWR0103
 U 1 1 5D7DD273
-P 8800 6250
-F 0 "#PWR0103" H 8800 6100 50  0001 C CNN
-F 1 "+3.3V" H 8815 6423 50  0000 C CNN
-F 2 "" H 8800 6250 50  0001 C CNN
-F 3 "" H 8800 6250 50  0001 C CNN
-	1    8800 6250
+P 3970 5460
+F 0 "#PWR0103" H 3970 5310 50  0001 C CNN
+F 1 "+3.3V" H 3985 5633 50  0000 C CNN
+F 2 "" H 3970 5460 50  0001 C CNN
+F 3 "" H 3970 5460 50  0001 C CNN
+	1    3970 5460
 	1    0    0    -1
 $EndComp
@@
 L power:PWR_FLAG #FLG0101
 U 1 1 5D7DD2FE
-P 8500 6250
-F 0 "#FLG0101" H 8500 6325 50  0001 C CNN
-F 1 "PWR_FLAG" H 8500 6424 50  0000 C CNN
-F 2 "" H 8500 6250 50  0001 C CNN
-F 3 "~" H 8500 6250 50  0001 C CNN
-	1    8500 6250
+P 3670 5460
+F 0 "#FLG0101" H 3670 5535 50  0001 C CNN
+F 1 "PWR_FLAG" H 3670 5634 50  0000 C CNN
+F 2 "" H 3670 5460 50  0001 C CNN
+F 3 "~" H 3670 5460 50  0001 C CNN
+	1    3670 5460
 	1    0    0    -1
 $EndComp
@@
 L power:+5V #PWR0104
 U 1 1 5D7DD3BD
-P 7750 6250
-F 0 "#PWR0104" H 7750 6100 50  0001 C CNN
-F 1 "+5V" H 7765 6423 50  0000 C CNN
-F 2 "" H 7750 6250 50  0001 C CNN
-F 3 "" H 7750 6250 50  0001 C CNN
-	1    7750 6250
+P 2920 5460
+F 0 "#PWR0104" H 2920 5310 50  0001 C CNN
+F 1 "+5V" H 2935 5633 50  0000 C CNN
+F 2 "" H 2920 5460 50  0001 C CNN
+F 3 "" H 2920 5460 50  0001 C CNN
+	1    2920 5460
 	1    0    0    -1
 $EndComp
@@
 L power:PWR_FLAG #FLG0102
 U 1 1 5D7DD3EB
-P 8050 6250
-F 0 "#FLG0102" H 8050 6325 50  0001 C CNN
-F 1 "PWR_FLAG" H 8050 6424 50  0000 C CNN
-F 2 "" H 8050 6250 50  0001 C CNN
-F 3 "~" H 8050 6250 50  0001 C CNN
-	1    8050 6250
-	1    0    0    -1
-$EndComp
-Wire Wire Line
-	8800 6250 8800 6400
-Wire Wire Line
-	8800 6400 8500 6400
-Wire Wire Line
-	8500 6400 8500 6250
-Wire Wire Line
-	8050 6250 8050 6400
-Wire Wire Line
-	8050 6400 7750 6400
-Wire Wire Line
-	7750 6400 7750 6250
+P 3220 5460
+F 0 "#FLG0102" H 3220 5535 50  0001 C CNN
+F 1 "PWR_FLAG" H 3220 5634 50  0000 C CNN
+F 2 "" H 3220 5460 50  0001 C CNN
+F 3 "~" H 3220 5460 50  0001 C CNN
+	1    3220 5460
+	1    0    0    -1
+$EndComp
+Wire Wire Line
+	3970 5460 3970 5610
+Wire Wire Line
+	3970 5610 3670 5610
+Wire Wire Line
+	3670 5610 3670 5460
+Wire Wire Line
+	3220 5460 3220 5610
+Wire Wire Line
+	3220 5610 2920 5610
+Wire Wire Line
+	2920 5610 2920 5460
 Wire Wire Line
 	5900 4150 5850 4150
@@
 L Mechanical:MountingHole H4
 U 1 1 5D803844
-P 7050 6550
-F 0 "H4" H 7150 6596 50  0000 L CNN
-F 1 "MountingHole" H 7150 6505 50  0000 L CNN
-F 2 "Mounting_Holes:MountingHole_2.7mm" H 7050 6550 50  0001 C CNN
-F 3 "~" H 7050 6550 50  0001 C CNN
-	1    7050 6550
+P 6920 4410
+F 0 "H4" H 7020 4456 50  0000 L CNN
+F 1 "MountingHole" H 7020 4365 50  0000 L CNN
+F 2 "Mounting_Holes:MountingHole_2.7mm" H 6920 4410 50  0001 C CNN
+F 3 "~" H 6920 4410 50  0001 C CNN
+	1    6920 4410
 	1    0    0    -1
 $EndComp
@@
 L Mechanical:MountingHole H3
 U 1 1 5D805BF3
-P 7050 6400
-F 0 "H3" H 7150 6446 50  0000 L CNN
-F 1 "MountingHole" H 7150 6355 50  0000 L CNN
-F 2 "Mounting_Holes:MountingHole_2.7mm" H 7050 6400 50  0001 C CNN
-F 3 "~" H 7050 6400 50  0001 C CNN
-	1    7050 6400
+P 6920 4260
+F 0 "H3" H 7020 4306 50  0000 L CNN
+F 1 "MountingHole" H 7020 4215 50  0000 L CNN
+F 2 "Mounting_Holes:MountingHole_2.7mm" H 6920 4260 50  0001 C CNN
+F 3 "~" H 6920 4260 50  0001 C CNN
+	1    6920 4260
 	1    0    0    -1
 $EndComp
@@
 L Mechanical:MountingHole H2
 U 1 1 5D805C29
-P 7050 6250
-F 0 "H2" H 7150 6296 50  0000 L CNN
-F 1 "MountingHole" H 7150 6205 50  0000 L CNN
-F 2 "Mounting_Holes:MountingHole_2.7mm" H 7050 6250 50  0001 C CNN
-F 3 "~" H 7050 6250 50  0001 C CNN
-	1    7050 6250
+P 6920 4110
+F 0 "H2" H 7020 4156 50  0000 L CNN
+F 1 "MountingHole" H 7020 4065 50  0000 L CNN
+F 2 "Mounting_Holes:MountingHole_2.7mm" H 6920 4110 50  0001 C CNN
+F 3 "~" H 6920 4110 50  0001 C CNN
+	1    6920 4110
 	1    0    0    -1
 $EndComp
@@
 L Mechanical:MountingHole H1
 U 1 1 5D805C61
-P 7050 6100
-F 0 "H1" H 7150 6146 50  0000 L CNN
-F 1 "MountingHole" H 7150 6055 50  0000 L CNN
-F 2 "Mounting_Holes:MountingHole_2.7mm" H 7050 6100 50  0001 C CNN
-F 3 "~" H 7050 6100 50  0001 C CNN
-	1    7050 6100
-	1    0    0    -1
-$EndComp
-Text Notes 7525 5375 0    50   ~ 0
-Optionally, can use 4.7k resistors instead of 10k (or vice versa).
+P 6920 3960
+F 0 "H1" H 7020 4006 50  0000 L CNN
+F 1 "MountingHole" H 7020 3915 50  0000 L CNN
+F 2 "Mounting_Holes:MountingHole_2.7mm" H 6920 3960 50  0001 C CNN
+F 3 "~" H 6920 3960 50  0001 C CNN
+	1    6920 3960
+	1    0    0    -1
+$EndComp
+Text Notes 3240 4400 0    50   ~ 0
+Optionally, can use 4.7k \nresistors instead of 10k \n(or vice versa).
 $Comp
 L Sensor_Temperature:DS1822 U4
